File: pcb/main/feeder2040.kicad_sch (KiCad schematic)
At the start: 80 parts, among them J1 USB4105-GF-A, J2 SWD_TagConnect, J3 Conn_ARM_JTAG_SWD_10, J4 0532610271, J5 0532610671, J6 009155005541006, SW1 1TS003B-2600-3500A-CT, SW2 1TS003B-2600-3500A-CT, SW3 1TS003B-2600-3500A-CT, SW4 1TS003B-2600-3500A-CT, U1 RP2040, U2 W25Q16JVUXIQ, U3 TPS62933DRLR, U4 AZ1117CH-3.3, U5 DRV8212PDSGR, U7 DRV8212PDSGR, U8 MAX3078EM/TR, Y1 12MHz

Commit message: First pass at routing complete
Parts:
- removed J3: Conn_ARM_JTAG_SWD_10, symbol Connector:Conn_ARM_JTAG_SWD_10
- removed JP1: SolderJumper_2_Open, symbol Jumper:SolderJumper_2_Open
- removed SW2: 1TS003B-2600-3500A-CT, symbol inventree:RIGHT ANGLE NO TACT SWITCH SMD,1.8x4.6mm
- added C33, C34: 100nF, Capacitor_SMD:C_0402_1005Metric, symbol inventree:50V 100nF X5R ±10% 0402
- added C35, C36: 2.2uF, Capacitor_SMD:C_0603_1608Metric, symbol inventree:CAP CER 2.2UF 50V X5R 0603
- added D4: B5819W, Diode_SMD:D_SOD-123, symbol inventree:DIODE SCHOTTKY 40V 1.5A SOD123FL
- added J7: Conn_ARM_SWD_TagConnect_TC2030-NL, Connector:Tag-Connect_TC2030-IDC-NL_2x03_P1.27mm_Vertical, symbol Connector:Conn_ARM_SWD_TagConnect_TC2030-NL
- added R25: 10kΩ, Resistor_SMD:R_0402_1005Metric, symbol inventree:RES 10K OHM 1% 1/16W 0402
- added R26, R27, R28, R29: 0Ω, Resistor_SMD:R_0402_1005Metric, symbol inventree:RES 0 OHM JUMPER 1/16W 0402
- added U6: DMG3415UQ-7, Package_TO_SOT_SMD:SOT-23-3, symbol inventree:MOSFET BVDSS 8V~24V SOT23 T&R 3
- C11, C7: footprint Capacitor_SMD:C_0603_1005Metric -> Capacitor_SMD:C_0603_1608Metric
- D1: footprint (none) -> Konkers_Diodes_LED:MEIHUA_MHS110FRGBCT
- D3: value SZMMSZ4684T1G -> MMSZ4684T1G
- J2: value SWD_TagConnect -> Conn_ARM_SWD_TagConnect_TC2030-NL
- J6: footprint (none) -> Konkers_Connectors_Header:AVX_009155005541006
- L1: footprint Inductor_SMD:L_12x12mm_H8mm -> Konkers_Inductors_SMD:Inductor_SMD_7.0mm_6.7mm_2.8mm; symbol inventree:FIXED IND 10UH 6.7A 19.5MOHM SMD -> inventree:FIXED IND 10UH 4A 67 MOHM SMD; ESR 19.5mΩ -> 67mΩ; IPN IND-000027-00 -> IND-000046-00; InvenTree 27 -> 46; Package Height 8.00mm -> 3.00mm; Package Size 12.00x12.00mm -> 7.00x6.60mm; Part URL /part/27/ -> /part/46/; Rated Current 6.7 A -> 4 A; Temperature Range -40~100°C -> -55~125°C
- R11: now left out of the parts list
- R7: now not fitted; now left out of the parts list
- SW1, SW3, SW4: footprint (none) -> Konkers_Mechanical_Switches:HYP_1TS003B_2600_3500A_CT
- U2: footprint (none) -> Konkers_Package_SON:USON-8-1EP_3x2mm_P0.5mm_EP0.3x1.7mm
- U4: value AZ1117CH-3.3 -> AZ1117CR-3.3; footprint Package_TO_SOT_SMD:SOT-223-3_TabPin2 -> Package_TO_SOT_SMD:SOT-89-3; symbol inventree:IC REG LINEAR 3.3V 1A SOT223 -> inventree:IC REG LINEAR 3.3V 1A SOT89; IPN PWR-000031-00 -> PWR-000047-00; InvenTree 31 -> 47; Package Type SOT-223-3 -> SOT-89-3; Part URL /part/31/ -> /part/47/
Connections:
- net +10V: now also C35.1, C36.1, D4.2 (A), R25.1, U6.1 (G); no longer C23.1, U4.3 (VI)
- net +1V1: now also U1.23 (DVDD), U1.45 (VREG_VOUT), U1.50 (DVDD)
- net +3V3: now also C33.2, C34.1, J7.1 (VCC); no longer U1.23 (DVDD), U1.45 (VREG_VOUT), U1.50 (DVDD)
- net BUTTON_FWD: now also U1.39 (GPIO27_ADC1)
- net BUTTON_REV: now also U1.40 (GPIO28_ADC2)
- net DRIVE_1: now also U1.29 (GPIO18)
- net DRIVE_2: now also U1.30 (GPIO19)
- net DRIVE_QUAD_A: now also U1.27 (GPIO16)
- net DRIVE_QUAD_B: now also U1.28 (GPIO17)
- net GND: now also J4.MP (MountPin), J5.MP (MountPin), J6.MP (MountPin), C33.1, C34.2, C35.2, C36.2, J7.5 (GND), R25.2, R26.1, R27.1, R28.2, R29.1
- net LED_B: now also U1.36 (GPIO24)
- net LED_G: now also U1.37 (GPIO25)
- net LED_R: now also U1.38 (GPIO26_ADC0)
- net MOTOR_EN: now also U1.31 (GPIO20)
- net ONE_WIRE: now also U1.17 (GPIO14)
- net PEEL_1: now also U1.34 (GPIO22)
- net PEEL_2: now also U1.35 (GPIO23)
- net PHOTON_RX: now also U1.16 (GPIO13)
- net PHOTON_RX_EN_N: now also U1.14 (GPIO11)
- net PHOTON_TX: now also U1.15 (GPIO12)
- net PHOTON_TX_EN: now also U1.13 (GPIO10)
- net QSPI_SCLK: now also U2.6 (CLK); no longer U2.7 (IO3)
- net QSPI_SD0: now also U2.5 (DI(IO0)); no longer U2.6 (CLK)
- net QSPI_SD1: now also U2.2 (DO(IO1)); no longer U2.5 (DI(IO0))
- net QSPI_SD2: now also U2.3 (IO2); no longer U2.2 (DO(IO1))
- net QSPI_SD3: now also U2.7 (IO3); no longer U2.3 (IO2)
- net RESET_N: now also J7.3 (~{RESET})
- net SWCLK: now also J7.4 (SWCLK)
- net SWD: now also J7.2 (SWDIO)
- net VBUS: now also U6.3 (D)
- net V24_PREFILTER: now reaches J6.1 (Pin_1), L2.2
- net at R7.1: now also U3.1 (RT)
- net 10V_SW: now reaches C15.2, L1.1, U3.5 (SW)
- net BOARD_ID_2: now reaches U1.11 (GPIO8)
- net BOARD_ID_2: now also R28.1
- net BOARD_ID_3: now reaches U1.12 (GPIO9)
- net BOARD_ID_3: now also R29.2
- net BOARD_ID_0: now reaches U1.5 (GPIO3)
- net BOARD_ID_0: now also R26.2
- net BOARD_ID_1: now reaches U1.6 (GPIO4)
- net BOARD_ID_1: now also R27.2
- net USBD_M renamed USBD_N
- new net REG_3V_INPUT: C23.1, D4.1 (K), U4.3 (VI), U6.2 (S)
- no-connect marks 5 -> 4
Other:
- moved on the sheet: C23, C24, C25, C26, C27, C28, L2, R19, SW3, U4, U5, U7
