File: pcb/main/cuttlefish-main.kicad_pcb (KiCad board)
At the start: 4 copper layers, 51.7 x 89 mm, 89 parts, among them J1 USB4105-GF-A, J2 Conn_ARM_SWD_TagConnect_TC203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, J4 0532610271, J5 0532610671, J6 009155005541006, J7 Conn_ARM_SWD_TagConnect_TC203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, SW1 1TS003B-2600-3500A-CT, SW3 1TS003B-2600-3500A-CT, SW4 1TS003B-2600-3500A-CT, U1 RP2040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

Commit message: Almost ready for rev0 fab
Parts:
- added G***: LOGO, Cuttlefish:cuttlefish, B.Cu at (141.7, 90.7)
Other:
- board text added: "copyright 2023 erik gilling github.com/konkers/cuttlefish rev ${REVISION}"
- board text added: "rev ${REVISION}"
