File: pcb/main/cuttlefish-main.kicad_sch (KiCad schematic)
At the start: 89 parts, among them J1 USB4105-GF-A, J2 Conn_ARM_SWD_TagConnect_TC203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, J4 0532610271, J5 0532610671, J6 009155005541006, J7 Conn_ARM_SWD_TagConnect_TC203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, SW1 1TS003B-2600-3500A-CT, SW3 1TS003B-2600-3500A-CT, SW4 1TS003B-2600-3500A-CT, U1 RP2040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

Commit message: Almost ready for rev0 fab
Parts:
- J2: value Conn_ARM_SWD_TagConnect_TC2030-NL -> ~
Connections:
- net BOARD_ID_2: now also R28.2; no longer R28.1
- net GND: now also R28.1; no longer R28.2
Other:
- note added: "10V Supply"
- note added: "3.3V Supply"
- note added: "BACK"
- note added: "Board ID"
- note added: "Bus Connector and Onewire Logic"
- note added: "Buttons"
- note added: "Drive Motor"
- note added: "FRONT"
- note added: "Indicator LED"
- note added: "Peel Motor"
- note added: "RP2040"
- note added: "RP2040 Decoupling"
- note added: "RP2040 Flash"
- note added: "RS485 Transceiver"
- note added: "SWD"
- note added: "USB-C 2.0 Port"
- moved on the sheet: C1, C10, C11, C12, C13, C14, C15, C16, C17, C18, C19, C2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
